File: design/BluetoothSpeakerKeyboard/BluetoothSpeakerKeyboard.kicad_pcb (KiCad board)
At the start: 2 copper layers, 50.4 x 15 mm, 13 parts, among them J1 Conn_01x06, SW1 BT_Key, SW2 V-, SW3 V+, SW4 start_pause

Commit message: adjustement and gerber files
Parts:
- C1: value 1uF -> 100nF; footprint Capacitor_SMD:C_0805_2012Metric -> Capacitor_SMD:C_0603_1608Metric_Pad1.08x0.95mm_HandSolder
- J1: footprint Connector_JST:JST_SH_BM06B-SRSS-TB_1x06-1MP_P1.00mm_Vertical -> Connector_JST:JST_SH_SM06B-SRSS-TB_1x06-1MP_P1.00mm_Horizontal
- R1, R2, R3: value 100k -> 1kΩ; footprint Resistor_SMD:R_0805_2012Metric -> Resistor_SMD:R_0402_1005Metric_Pad0.72x0.64mm_HandSolder
- R4, R5, R6, R7: value R -> 1kΩ; footprint Resistor_SMD:R_0805_2012Metric -> Resistor_SMD:R_0402_1005Metric_Pad0.72x0.64mm_HandSolder
- moved J1 0.59 mm to (61.4, 23.5), turned to 180 degrees
Routing:
- net Net-(J1-Pin_6): track 44.7 -> 43.4 mm
- net Net-(J1-Pin_2): track 48.4 -> 47.1 mm
- net Net-(J1-Pin_3): track 35.5 -> 34.8 mm
