File: design/BluetoothSpeakerKeyboard/BluetoothSpeakerKeyboard.kicad_sch (KiCad schematic)
At the start: 13 parts, among them J1 Conn_01x06, SW1 BT_Key, SW2 V-, SW3 V+, SW4 start_pause

Commit message: adjustement and gerber files
Parts:
- C1: value 1uF -> 100nF; footprint Capacitor_SMD:C_0805_2012Metric -> Capacitor_SMD:C_0603_1608Metric_Pad1.08x0.95mm_HandSolder
- J1: footprint Connector_JST:JST_SH_BM06B-SRSS-TB_1x06-1MP_P1.00mm_Vertical -> Connector_JST:JST_SH_SM06B-SRSS-TB_1x06-1MP_P1.00mm_Horizontal
- R1, R2, R3: value 100k -> 1kΩ; footprint Resistor_SMD:R_0805_2012Metric -> Resistor_SMD:R_0402_1005Metric_Pad0.72x0.64mm_HandSolder
- R4, R5, R6, R7: value R -> 1kΩ; footprint Resistor_SMD:R_0805_2012Metric -> Resistor_SMD:R_0402_1005Metric_Pad0.72x0.64mm_HandSolder
Changed lines of the file:
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@@
 			)
 		)
-		(property "Value" "100k"
+		(property "Value" "1kΩ"
 			(at 110.49 59.944 90)
 			(effects
@@
 			)
 		)
-		(property "Footprint" "Resistor_SMD:R_0805_2012Metric"
+		(property "Footprint" "Resistor_SMD:R_0402_1005Metric_Pad0.72x0.64mm_HandSolder"
 			(at 110.49 58.928 90)
 			(effects
@@
 			)
 		)
-		(property "Value" "1uF"
+		(property "Value" "100nF"
 			(at 96.52 51.562 0)
 			(effects
@@
 			)
 		)
-		(property "Footprint" "Capacitor_SMD:C_0805_2012Metric"
+		(property "Footprint" "Capacitor_SMD:C_0603_1608Metric_Pad1.08x0.95mm_HandSolder"
 			(at 102.5652 58.42 0)
 			(effects
@@
 			)
 		)
-		(property "Value" "100k"
+		(property "Value" "1kΩ"
 			(at 110.49 44.196 90)
 			(effects
@@
 			)
 		)
-		(property "Footprint" "Resistor_SMD:R_0805_2012Metric"
+		(property "Footprint" "Resistor_SMD:R_0402_1005Metric_Pad0.72x0.64mm_HandSolder"
 			(at 110.49 43.688 90)
 			(effects
@@
 			)
 		)
-		(property "Value" "100k"
+		(property "Value" "1kΩ"
 			(at 110.49 51.816 90)
 			(effects
@@
 			)
 		)
-		(property "Footprint" "Resistor_SMD:R_0805_2012Metric"
+		(property "Footprint" "Resistor_SMD:R_0402_1005Metric_Pad0.72x0.64mm_HandSolder"
 			(at 110.49 51.308 90)
 			(effects
@@
 			)
 		)
-		(property "Value" "R"
+		(property "Value" "1kΩ"
 			(at 92.71 80.772 90)
 			(effects
@@
 			)
 		)
-		(property "Footprint" "Resistor_SMD:R_0805_2012Metric"
+		(property "Footprint" "Resistor_SMD:R_0402_1005Metric_Pad0.72x0.64mm_HandSolder"
 			(at 92.71 80.518 90)
 			(effects
@@
 			)
 		)
-		(property "Value" "R"
+		(property "Value" "1kΩ"
 			(at 92.71 60.452 90)
 			(effects
@@
 			)
 		)
-		(property "Footprint" "Resistor_SMD:R_0805_2012Metric"
+		(property "Footprint" "Resistor_SMD:R_0402_1005Metric_Pad0.72x0.64mm_HandSolder"
 			(at 92.71 60.198 90)
 			(effects
@@
 			)
 		)
-		(property "Value" "R"
+		(property "Value" "1kΩ"
 			(at 92.71 101.346 90)
 			(effects
@@
 			)
 		)
-		(property "Footprint" "Resistor_SMD:R_0805_2012Metric"
+		(property "Footprint" "Resistor_SMD:R_0402_1005Metric_Pad0.72x0.64mm_HandSolder"
 			(at 92.71 100.838 90)
 			(effects
@@
 			)
 		)
-		(property "Footprint" "Connector_JST:JST_SH_BM06B-SRSS-TB_1x06-1MP_P1.00mm_Vertical"
+		(property "Footprint" "Connector_JST:JST_SH_SM06B-SRSS-TB_1x06-1MP_P1.00mm_Horizontal"
 			(at 157.48 71.12 0)
 			(effects
@@
 			)
 		)
-		(property "Value" "R"
+		(property "Value" "1kΩ"
 			(at 92.71 118.872 90)
 			(effects
@@
 			)
 		)
-		(property "Footprint" "Resistor_SMD:R_0805_2012Metric"
+		(property "Footprint" "Resistor_SMD:R_0402_1005Metric_Pad0.72x0.64mm_HandSolder"
 			(at 92.71 118.618 90)
 			(effects
